File: MC34063_buck/MC34063_buck.sch (KiCad schematic (older format))
At the start: 23 parts, among them J1 INPUT, J2 OUTPUT, Q1 2N2222, U1 MC34063AP

Commit message: Gerbers
Parts:
- C2: value 100p -> 22p
- L1: value 10u -> 100u
Changed lines of the file:
@@
 P 5450 3150
 F 0 "L1" H 5502 3196 50  0000 L CNN
-F 1 "10u" H 5502 3105 50  0000 L CNN
+F 1 "100u" H 5502 3105 50  0000 L CNN
 F 2 "Inductor_THT:L_Radial_D10.0mm_P5.00mm_Neosid_SD12k_style3" H 5450 3150 50  0001 C CNN
 F 3 "~" H 5450 3150 50  0001 C CNN
@@
 P 3350 3450
 F 0 "C2" H 3465 3496 50  0000 L CNN
-F 1 "100p" H 3465 3405 50  0000 L CNN
+F 1 "22p" H 3465 3405 50  0000 L CNN
 F 2 "Capacitor_THT:C_Disc_D7.0mm_W2.5mm_P5.00mm" H 3388 3300 50  0001 C CNN
 F 3 "~" H 3350 3450 50  0001 C CNN
